File: elec/layout/default/mt6701.kicad_pcb (KiCad board)
At the start: 2 copper layers, 225.7 x 100.8 mm, 0 parts

Commit message: added default layout
Parts:
- added C1: 50V 100nF X7R ±10% 0603 Multilayer Ceramic Capacitors MLCC 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, lib:C0603, F.Cu at (240.1, 99.4)
- added U1: , lib:SOP-8_L4.9-W3.9-P1.27-LS6.0-BL, F.Cu at (238.8, 95.6)
Routing:
- net gnd: track 0.00 -> 7.41 mm
- net vcc: track 0.00 -> 3.43 mm
Changed lines of the file:
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@@
   )
   (net 0 "")
+  (net 1 "vcc")
+  (net 2 "out")
+  (net 3 "gnd")
+  (net 4 "z")
+  (net 5 "b")
+  (net 6 "a")
+  (net 7 "push")
+  (footprint "lib:C0603" (layer "F.Cu")
+    (at 240.08 99.4 180)
+    (descr "Capacitor SMD 0603 (1608 Metric), square (rectangular) end terminal, IPC_7351 nominal, (Body size source: IPC-SM-782 page 76, https://www.pcb-3d.com/wordpress/wp-content/uploads/ipc-sm-782a_amendment_1_and_2.pdf), generated with kicad-footprint-generator")
+    (tags "capacitor")
+    (attr smd)
+    (fp_text reference "C1" (at 0 -1.43) (layer "F.SilkS")
+        (effects (font (size 1 1) (thickness 0.15)))
+    )
+    (fp_text value "50V 100nF X7R ±10% 0603  Multilayer Ceramic Capacitors MLCC - SMD/SMT ROHS" (at 0.08 -3) (layer "F.Fab")
+        (effects (font (size 1 1) (thickness 0.15)))
+    )
+    (fp_text user "${REFERENCE}" (at 0 0) (layer "F.Fab")
+        (effects (font (size 0.4 0.4) (thickness 0.06)))
+    )
+    (fp_line (start -0.14058 -0.51) (end 0.14058 -0.51)
+      (stroke (width 0.12) (type solid)) (layer "F.SilkS"))
+    (fp_line (start -0.14058 0.51) (end 0.14058 0.51)
+      (stroke (width 0.12) (type solid)) (layer "F.SilkS"))
+    (fp_line (start -1.48 -0.73) (end 1.48 -0.73)
+      (stroke (width 0.05) (type solid)) (layer "F.CrtYd"))
+    (fp_line (start -1.48 0.73) (end -1.48 -0.73)
+      (stroke (width 0.05) (type solid)) (layer "F.CrtYd"))
+    (fp_line (start 1.48 -0.73) (end 1.48 0.73)
+      (stroke (width 0.05) (type solid)) (layer "F.CrtYd"))
+    (fp_line (start 1.48 0.73) (end -1.48 0.73)
+      (stroke (width 0.05) (type solid)) (layer "F.CrtYd"))
+    (fp_line (start -0.8 -0.4) (end 0.8 -0.4)
+      (stroke (width 0.1) (type solid)) (layer "F.Fab"))
+    (fp_line (start -0.8 0.4) (end -0.8 -0.4)
+      (stroke (width 0.1) (type solid)) (layer "F.Fab"))
+    (fp_line (start 0.8 -0.4) (end 0.8 0.4)
+      (stroke (width 0.1) (type solid)) (layer "F.Fab"))
+    (fp_line (start 0.8 0.4) (end -0.8 0.4)
+      (stroke (width 0.1) (type solid)) (layer "F.Fab"))
+    (pad "1" smd roundrect (at -0.775 0 180) (size 0.9 0.95) (layers "F.Cu" "F.Paste" "F.Mask") (roundrect_rratio 0.25)
+      (net 1 "vcc") (pintype "stereo"))
+    (pad "2" smd roundrect (at 0.775 0 180) (size 0.9 0.95) (layers "F.Cu" "F.Paste" "F.Mask") (roundrect_rratio 0.25)
+      (net 3 "gnd") (pintype "stereo"))
+    (model "${KICAD6_3DMODEL_DIR}/Capacitor_SMD.3dshapes/C_0603_1608Metric.wrl"
+      (offset (xyz 0 0 0))
+      (scale (xyz 1 1 1))
+      (rotate (xyz 0 0 0))
+    )
+  )
+  (footprint "lib:SOP-8_L4.9-W3.9-P1.27-LS6.0-BL" (layer "F.Cu")
+    (at 238.8 95.6 90)
+    (attr smd)
+    (fp_text reference "U1" (at 0 -6.68 90) (layer "F.SilkS")
+        (effects (font (size 1 1) (thickness 0.15)))
+    )
+    (fp_text value "" (at 0 6.68 90) (layer "F.Fab")
+        (effects (font (size 1 1) (thickness 0.15)))
+    )
+    (fp_text user "${REFERENCE}" (at 0 0 90) (layer "F.Fab")
+        (effects (font (size 1 1) (thickness 0.15)))
+    )
+    (fp_line (start -2.58 -1.52) (end 2.58 -1.52)
+      (stroke (width 0.15) (type solid)) (layer "F.SilkS"))
+    (fp_line (start -2.58 1.52) (end -2.58 -1.52)
+      (stroke (width 0.15) (type solid)) (layer "F.SilkS"))
+    (fp_line (start 2.58 -1.52) (end 2.58 1.52)
+      (stroke (width 0.15) (type solid)) (layer "F.SilkS"))
+    (fp_line (start 2.58 1.52) (end -2.58 1.52)
+      (stroke (width 0.15) (type solid)) (layer "F.SilkS"))
+    (fp_circle (center -2.67 2.68) (end -2.52 2.68)
+      (stroke (width 0.3) (type solid)) (fill none) (layer "F.SilkS"))
+    (fp_circle (center -1.91 0.77) (end -1.76 0.77)
+      (stroke (width 0.3) (type solid)) (fill none) (layer "F.SilkS"))
+    (fp_circle (center -1.91 3.4) (end -1.76 3.4)
+      (stroke (width 0.3) (type solid)) (fill none) (layer "Cmts.User"))
+    (fp_circle (center -2.45 3) (end -2.42 3)
+      (stroke (width 0.06) (type solid)) (fill none) (layer "F.Fab"))
+    (pad "1" smd oval (at -1.91 2.68 90) (size 0.63 1.86) (layers "F.Cu" "F.Paste" "F.Mask")
+      (net 1 "vcc") (pintype "stereo"))
+    (pad "2" smd oval (at -0.63 2.68 90) (size 0.63 1.86) (layers "F.Cu" "F.Paste" "F.Mask")
+      (net 1 "vcc") (pintype "stereo"))
+    (pad "3" smd oval (at 0.63 2.68 90) (size 0.63 1.86) (layers "F.Cu" "F.Paste" "F.Mask")
+      (net 2 "out") (pintype "stereo"))
+    (pad "4" smd oval (at 1.9 2.68 90) (size 0.63 1.86) (layers "F.Cu" "F.Paste" "F.Mask")
+      (net 3 "gnd") (pintype "stereo"))
+    (pad "5" smd oval (at 1.9 -2.68 90) (size 0.63 1.86) (layers "F.Cu" "F.Paste" "F.Mask")
+      (net 7 "push") (pintype "stereo"))
+    (pad "6" smd oval (at 0.63 -2.68 90) (size 0.63 1.86) (layers "F.Cu" "F.Paste" "F.Mask")
+      (net 6 "a") (pintype "stereo"))
+    (pad "7" smd oval (at -0.63 -2.68 90) (size 0.63 1.86) (layers "F.Cu" "F.Paste" "F.Mask")
+      (net 5 "b") (pintype "stereo"))
+    (pad "8" smd oval (at -1.91 -2.68 90) (size 0.63 1.86) (layers "F.Cu" "F.Paste" "F.Mask")
+      (net 4 "z") (pintype "stereo"))
+    (model "/Users/nickk/projects/chess-clock/.ato/modules/smart-knob/.ato/modules/mt6701/elec/footprints/footprints.3dshapes/SOP-8_L4.9-W3.9-P1.27-LS6.0-BL-1.wrl"
+      (offset (xyz 0 -0 -0))
+      (scale (xyz 1 1 1))
+      (rotate (xyz 0 0 0))
+    )
+  )
   (gr_circle (center 225.62 81.79) (end 227.32 81.79)
     (stroke (width 0.1) (type solid)) (fill none) (layer "Edge.Cuts"))
@@
       (xy 69.100734 49.778315)
     )
-    (stroke (width 0) (type solid)) (fill none) (layer "Edge.Cuts"))
+    (stroke (width 0.1) (type solid)) (fill none) (layer "Edge.Cuts"))
   (gr_arc (start 261.62 113.79) (mid 260.448427 116.618427) (end 257.62 117.79)
     (stroke (width 0.1) (type solid)) (layer "Edge.Cuts"))
@@
     (effects (font (size 2 2) (thickness 0.1)) (justify left bottom))
   )
+  (segment (start 241 96.71) (end 241.48 96.23) (width 0.25) (layer "F.Cu") (net 1))
+  (segment (start 240.855 99.4) (end 241 99.255) (width 0.25) (layer "F.Cu") (net 1))
+  (segment (start 241 99.255) (end 241 96.71) (width 0.25) (layer "F.Cu") (net 1))
+  (segment (start 240.1 93.7) (end 239.6 94.2) (width 0.25) (layer "F.Cu") (net 3))
+  (segment (start 239.6 99.105) (end 239.305 99.4) (width 0.25) (layer "F.Cu") (net 3))
+  (segment (start 239.6 94.2) (end 239.6 99.105) (width 0.25) (layer "F.Cu") (net 3))
+  (segment (start 241.48 93.7) (end 240.1 93.7) (width 0.25) (layer "F.Cu") (net 3))
   (group "" (id 6c1ef9f7-0f34-47bb-ac1a-76df23fb396e)
     (members
